Commit message: Changes: *the PosePub is added which can publish the pose of any objects in gazebo to ros topics has multiple uses in this project Bugs ;
* auto rotating robot problem encountered
fix: adjusting mu mu1 values accordingly

To do:
* reward function
* sensor for publishing the nearest obs distances
* fix the bug
* directionality test

File: mybot_ws/src/mybot_description/urdf/mybot.xacro (robot description, xacro)
@@ -75,5 +75,5 @@
   <link name="left_wheel">
     <!--origin xyz="0.1 0.13 0.1" rpy="0 1.5707 1.5707"/-->
-    <collision name="collision">
+    <collision name="collision_left">
       <origin xyz="0 0 0" rpy="0 1.5707 1.5707"/>
       <geometry>
@@ -87,4 +87,14 @@
       </geometry>
     </visual>
+     <surface>
+        <friction>
+          <ode>
+            <mu>0.1</mu>
+            <mu2>0.1</mu2>
+            <slip1>0</slip1>
+            <slip2>0</slip2>
+          </ode>
+        </friction>
+      </surface>
     <inertial>
       <origin xyz="0 0 0" rpy="0 1.5707 1.5707"/>
@@ -110,4 +120,14 @@
       </geometry>
     </visual>
+     <surface>
+        <friction>
+          <ode>
+            <mu>0.1</mu>
+            <mu2>0.1</mu2>
+            <slip1>0</slip1>
+            <slip2>0</slip2>
+          </ode>
+        </friction>
+      </surface>
     <inertial>
       <origin xyz="0 0 0" rpy="0 1.5707 1.5707"/>
@@ -170,4 +190,12 @@
     <child link="hokuyo"/>
   </joint>
+<!-- eagle is link planeed to introduced for getting the nearest obstacle dist to design the reward function -->
+<!-- planning to introduce it later after some more reasearch in open ai Ros Gazebo libaries -->
+  <!-- <joint name="eagle_joint" type="fixed">
+    <axis xyz="0 1 0" />
+    <origin xyz=".15 -0.5 .1" rpy="0 0 0"/>
+    <parent link="chassis"/>
+    <child link="eagle"/>
+  </joint> -->
   <!-- Hokuyo Laser -->
   <link name="hokuyo">
@@ -190,3 +218,22 @@
     </inertial>
   </link>
+<!-- <link name="eagle">
+    <collision>
+      <origin xyz="0 0 0" rpy="0 0 0"/>
+      <geometry>
+    <box size="0.1 0.1 0.1"/>
+      </geometry>
+    </collision>
+    <visual>
+      <origin xyz="0 0 0" rpy="0 0 0"/>
+      <geometry>
+        <mesh filename="package://mybot_description/meshes/hokuyo.dae"/>
+      </geometry>
+    </visual>
+    <inertial>
+      <mass value="1e-5" />
+      <origin xyz="0 0 0" rpy="0 0 0"/>
+      <inertia ixx="1e-6" ixy="0" ixz="0" iyy="1e-6" iyz="0" izz="1e-6" />
+    </inertial>
+  </link> -->
 </robot>

Commit message: the changes are to done to code to check the posepub and setpose packages to debug errors - the directionality test env is setup to test the energy waveform against angle of incidence - the interias and friction components for wheel were changed BUGS :: - the batbot is still suspectble to automatic rotation along the z axis and contact points in the wheel seems jittery - have to change the friction and interias to get out of it

File: mybot_ws/src/mybot_description/urdf/mybot.xacro (robot description, xacro)
@@ -9,6 +9,6 @@
     <pose>0 0 0.1 0 0 0</pose>
     <inertial>
-      <mass value="15.0"/>
-      <origin xyz="0.0 0 0.1" rpy=" 0 0 0"/>
+      <mass value="15.00"/>
+      <origin xyz="0.0 0 0.0" rpy=" 0 0 0"/>
       <inertia
           ixx="0.1" ixy="0" ixz="0"
@@ -66,6 +66,14 @@
       </surface>
     </collision>
+    <!-- <inertial>
+      <origin xyz="0 0 0" rpy="0 1.5707 1.5707"/>
+      <mass value="1"/>
+      <interia
+        ixx=".01" ixy="0.0" ixz="0.0"
+        iyy=".01" iyz="0.0"
+        izz=".01"/>
+    </inertial> -->
     <visual name='caster_front_visual'>
-      <origin xyz="0.15 0 -0.05" rpy=" 0 0 0"/>
+      <origin xyz="0.15 0 -0.06" rpy=" 0 0 0"/>
       <geometry>
         <sphere radius="0.05"/>
@@ -80,28 +88,28 @@
         <cylinder radius="0.1" length="0.05"/>
       </geometry>
-    </collision>
-    <visual name="left_wheel_visual">
-      <origin xyz="0 0 0" rpy="0 1.5707 1.5707"/>
-      <geometry>
-        <cylinder radius="0.1" length="0.05"/>
-      </geometry>
-    </visual>
-     <surface>
-        <friction>
-          <ode>
-            <mu>0.1</mu>
-            <mu2>0.1</mu2>
+      <!-- <surface>
+        <friction>
+          <ode>
+            <mu>10000.0</mu>
+            <mu2>10000.0</mu2>
             <slip1>0</slip1>
             <slip2>0</slip2>
           </ode>
         </friction>
-      </surface>
-    <inertial>
-      <origin xyz="0 0 0" rpy="0 1.5707 1.5707"/>
+      </surface> -->
+    </collision>
+    <visual name="left_wheel_visual">
+      <origin xyz="0 0 0" rpy="0 1.5707 1.5707"/>
+      <geometry>
+        <cylinder radius="0.1" length="0.05"/>
+      </geometry>
+    </visual>
+    <inertial>
+      <origin xyz="0 -0.0 0" rpy="0 1.5707 1.5707"/>
       <mass value="5"/>
       <inertia
-        ixx=".1" ixy="0.0" ixz="0.0"
-        iyy=".1" iyz="0.0"
-        izz=".1"/>
+        ixx=".01" ixy="0.0" ixz="0.0"
+        iyy=".01" iyz="0.0"
+        izz=".01"/>
     </inertial>
   </link>
@@ -113,28 +121,28 @@
         <cylinder radius="0.1" length="0.05"/>
       </geometry>
-    </collision>
-    <visual name="right_wheel_visual">
-      <origin xyz="0 0 0" rpy="0 1.5707 1.5707"/>
-      <geometry>
-        <cylinder radius="0.1" length="0.05"/>
-      </geometry>
-    </visual>
-     <surface>
-        <friction>
-          <ode>
-            <mu>0.1</mu>
-            <mu2>0.1</mu2>
+      <!-- <surface>
+        <friction>
+          <ode>
+            <mu>10000.0</mu>
+            <mu2>10000.0</mu2>
             <slip1>0</slip1>
             <slip2>0</slip2>
           </ode>
         </friction>
-      </surface>
-    <inertial>
-      <origin xyz="0 0 0" rpy="0 1.5707 1.5707"/>
+      </surface> -->
+    </collision>
+    <visual name="right_wheel_visual">
+      <origin xyz="0 0 0" rpy="0 1.5707 1.5707"/>
+      <geometry>
+        <cylinder radius="0.1" length="0.05"/>
+      </geometry>
+    </visual>
+    <inertial>
+      <origin xyz="0 0.0 0" rpy="0 1.5707 1.5707"/>
       <mass value="5"/>
       <inertia
-        ixx=".1" ixy="0.0" ixz="0.0"
-        iyy=".1" iyz="0.0"
-        izz=".1"/>
+        ixx=".01" ixy="0.0" ixz="0.0"
+        iyy=".01" iyz="0.0"
+        izz=".01"/>
     </inertial>
   </link>

Commit message: the check.py was modified to calulate the directionality data -- time sync is been applied to the msgs :: --- bugs--- * interia error causes the robot movements * python3 not working with msg_filter lib missing python3 distpackages ---- to do--- * new robot model * action script for robot movementes * open-ai gym ros interface script * directionality graph * RL design

File: mybot_ws/src/mybot_description/urdf/mybot.xacro (robot description, xacro)
@@ -3,4 +3,31 @@
   <xacro:property name="cameraSize" value="0.05"/>
   <xacro:property name="cameraMass" value="0.1"/>
+  <xacro:property name = "chassisMass" value = "15.00"/>
+  <xacro:property name = "chassisX" value = "0.4"/>
+  <xacro:property name = "chassisY" value = "0.2"/>
+  <xacro:property name = "chassisZ" value = "0.1"/>
+  <xacro:property name = "wheelMass" value = "5.00"/>
+  <xacro:property name = "wheelR" value = "0.1"/>
+  <xacro:property name = "wheelH" value = "0.05"/>
+  <xacro:property name = "castorMass" value = "5.00"/>
+  <xacro:property name = "castorRadius" value = "0.05"/>
+  <!-- macro name="cylinder_inertia" params="m r h">
+    <inertia  ixx="${m*(3*r*r+h*h)/12}" ixy = "0" ixz = "0"
+      iyy="${m*(3*r*r+h*h)/12}" iyz = "0"
+      izz="${m*r*r/2}"
+    />
+  </macro>
+  <macro name="box_inertia" params="m x y z">
+    <inertia  ixx="${m*(y*y+z*z)/12}" ixy = "0" ixz = "0"
+      iyy="${m*(x*x+z*z)/12}" iyz = "0"
+      izz="${m*(x*x+z*z)/12}"
+    />
+  </macro>
+  <macro name="sphere_inertia" params="m r">
+    <inertia  ixx="${2*m*r*r/5}" ixy = "0" ixz = "0"
+      iyy="${2*m*r*r/5}" iyz = "0"
+      izz="${2*m*r*r/5}"
+    />
+  </macro>  -->
   <xacro:include filename="$(find mybot_description)/urdf/mybot.gazebo" />
   <xacro:include filename="$(find mybot_description)/urdf/materials.xacro" />
@@ -9,10 +36,10 @@
     <pose>0 0 0.1 0 0 0</pose>
     <inertial>
-      <mass value="15.00"/>
+      <mass value="${chassisMass}"/>
       <origin xyz="0.0 0 0.0" rpy=" 0 0 0"/>
       <inertia
-          ixx="0.1" ixy="0" ixz="0"
-          iyy="0.1" iyz="0"
-          izz="0.1"
+          ixx="${chassisMass*(chassisY*chassisY*chassisZ*chassisZ)/12}" ixy="0" ixz="0"
+          iyy="${chassisMass*(chassisX*chassisX*chassisZ*chassisZ)/12}" iyz="0"
+          izz="${chassisMass*(chassisX*chassisX*chassisY*chassisY)/12}"
       />
     </inertial>
@@ -31,5 +58,5 @@
       <origin xyz="-0.15 0 -0.05" rpy=" 0 0 0"/>
       <geometry>
-        <sphere radius="0.05"/>
+        <sphere radius="${castorRadius}"/>
       </geometry>
       <surface>
@@ -47,5 +74,5 @@
       <origin xyz="-0.15 0 -0.05" rpy=" 0 0 0"/>
       <geometry>
-        <sphere radius="0.05"/>
+        <sphere radius="${castorRadius}"/>
       </geometry>
     </visual>
@@ -53,5 +80,5 @@
       <origin xyz="0.15 0 -0.05" rpy=" 0 0 0"/>
       <geometry>
-        <sphere radius="0.05"/>
+        <sphere radius="${castorRadius}"/>
       </geometry>
       <surface>
@@ -77,8 +104,12 @@
       <origin xyz="0.15 0 -0.06" rpy=" 0 0 0"/>
       <geometry>
-        <sphere radius="0.05"/>
-      </geometry>
-    </visual>
-  </link>
+        <sphere radius="${castorRadius}"/>
+      </geometry>
+    </visual>
+  </link>
+ <!-- <inertia  ixx="${m*(3*r*r+h*h)/12}" ixy = "0" ixz = "0"
+      iyy="${m*(3*r*r+h*h)/12}" iyz = "0"
+      izz="${m*r*r/2}"
+    /> -->
   <link name="left_wheel">
     <!--origin xyz="0.1 0.13 0.1" rpy="0 1.5707 1.5707"/-->
@@ -86,5 +117,5 @@
       <origin xyz="0 0 0" rpy="0 1.5707 1.5707"/>
       <geometry>
-        <cylinder radius="0.1" length="0.05"/>
+        <cylinder radius="${wheelR}" length="${wheelH}"/>
       </geometry>
       <!-- <surface>
@@ -102,14 +133,14 @@
       <origin xyz="0 0 0" rpy="0 1.5707 1.5707"/>
       <geometry>
-        <cylinder radius="0.1" length="0.05"/>
+        <cylinder radius="${wheelR}" length="${wheelH}"/>
       </geometry>
     </visual>
     <inertial>
       <origin xyz="0 -0.0 0" rpy="0 1.5707 1.5707"/>
-      <mass value="5"/>
+      <mass value="${wheelMass}"/>
       <inertia
-        ixx=".01" ixy="0.0" ixz="0.0"
-        iyy=".01" iyz="0.0"
-        izz=".01"/>
+        ixx="${wheelMass * (3 * wheelR * wheelR + wheelH * wheelH)/12}" ixy="0.0" ixz="0.0"
+        iyy="${wheelMass * (3 * wheelR * wheelR + wheelH * wheelH)/12}" iyz="0.0"
+        izz="${wheelMass * (3 * wheelR * wheelR + wheelH * wheelH)/12}"/>
     </inertial>
   </link>
@@ -119,5 +150,5 @@
       <origin xyz="0 0 0" rpy="0 1.5707 1.5707"/>
       <geometry>
-        <cylinder radius="0.1" length="0.05"/>
+        <cylinder radius="${wheelR}" length="${wheelH}"/>
       </geometry>
       <!-- <surface>
@@ -135,14 +166,14 @@
       <origin xyz="0 0 0" rpy="0 1.5707 1.5707"/>
       <geometry>
-        <cylinder radius="0.1" length="0.05"/>
-      </geometry>
-    </visual>
-    <inertial>
-      <origin xyz="0 0.0 0" rpy="0 1.5707 1.5707"/>
-      <mass value="5"/>
+       <cylinder radius="${wheelR}" length="${wheelH}"/>
+      </geometry>
+    </visual>
+     <inertial>
+      <origin xyz="0 -0.0 0" rpy="0 1.5707 1.5707"/>
+      <mass value="${wheelMass}"/>
       <inertia
-        ixx=".01" ixy="0.0" ixz="0.0"
-        iyy=".01" iyz="0.0"
-        izz=".01"/>
+        ixx="${wheelMass * (3 * wheelR * wheelR + wheelH * wheelH)/12}" ixy="0.0" ixz="0.0"
+        iyy="${wheelMass * (3 * wheelR * wheelR + wheelH * wheelH)/12}" iyz="0.0"
+        izz="${wheelMass * (3 * wheelR * wheelR + wheelH * wheelH)/12}"/>
     </inertial>
   </link>

Commit message: -----changes---- check.py was modified to accomate polar cloud (3d-points) *the sonar_gen was modefied to include in lib python * mybot.xacro wad modified to remove the interia bugs --bugs-- * python3 error was solved by using python2.7 for every files * interia error was solved approx increasing the param from 0.1 to 0.2 * more testing needs to done * reinstalling ros-gazebo might have lost some packages --to do-- * new robot model     * action script for robot movementes     * open-ai gym ros interface script     * directionality graph * RL design

File: mybot_ws/src/mybot_description/urdf/mybot.xacro (robot description, xacro)
@@ -3,5 +3,5 @@
   <xacro:property name="cameraSize" value="0.05"/>
   <xacro:property name="cameraMass" value="0.1"/>
-  <xacro:property name = "chassisMass" value = "15.00"/>
+  <xacro:property name = "chassisMass" value = "10.00"/>
   <xacro:property name = "chassisX" value = "0.4"/>
   <xacro:property name = "chassisY" value = "0.2"/>
@@ -38,9 +38,19 @@
       <mass value="${chassisMass}"/>
       <origin xyz="0.0 0 0.0" rpy=" 0 0 0"/>
-      <inertia
+      <!-- <inertia
           ixx="${chassisMass*(chassisY*chassisY*chassisZ*chassisZ)/12}" ixy="0" ixz="0"
           iyy="${chassisMass*(chassisX*chassisX*chassisZ*chassisZ)/12}" iyz="0"
           izz="${chassisMass*(chassisX*chassisX*chassisY*chassisY)/12}"
+      /> -->
+   <inertia
+          ixx="0.2" ixy="0" ixz="0"
+          iyy="0.2" iyz="0"
+          izz="0.2"
       />
+      <!-- <box_inertia
+				m="${chassisMass}"
+				x="${chassisX}"
+				y="${chassisY}"
+				z="${chassisZ}"/> -->
     </inertial>
     <collision name='collision'>
